Commit message: URDF devam

File: Notlar/URDF_Dosyasi_Olusturma/simple_robot.urdf (robot description, URDF)
Before this commit: robot simple_robot, 1 links, 0 joints
Links:
- link base_link: geometry visual box size=0.5 0.5 0.5

Commit message: URDF bölümü tamamlandı.

File: Notlar/URDF_Dosyasi_Olusturma/simple_robot.urdf (robot description, URDF)
Before this commit: robot simple_robot, 1 links, 0 joints
Links:
- added link second_link; visual cylinder length=0.15 radius=0.25
Joints:
- added joint bazse_second_joint: type fixed, parent base_link, child second_link, origin xyz=0.5 0 0 rpy=0 0 0
