Commit message: Kendimiz başlatabileceğimiz şekilde klasörleme ve gerekli kodlamalar yapılıyor. Devam edilecek.

File: Projeler/Robot_Modelleme/src/my_robot_description/urdf/my_robot.urdf (robot description, URDF)
Before this commit: robot my_robot, 2 links, 3 joints
Links:
- added link base_footprint
Joints:
- added joint base_joint: type fixed, parent base_footprint, child base_link, origin xyz=0 0 ${(base_height/2)+wheel_radius} rpy=0.0 0.0 0.0
