Commit message: Klasörleme ile kod sadeleştirme işlemi gerçekleştirildi.

File: Projeler/Robot_Modelleme/src/my_robot_description/urdf/my_robot.xacro (robot description, xacro)
@@ -1,10 +1,4 @@
 <?xml version="1.0"?>
 <robot name="my_robot" xmlns:xacro = "http://www.ros.org/wiki/xacro>" > <!-- xmlns:xacro = "http://www.ros.org/wiki/xacro>" kısmı xacro kullanabilmek için.-->
-    <material name="cyan">
-        <color rgba="0 1 1 1"/>
-    </material>
-    <material name="black">
-        <color rgba="0 0 0 1"/>
-    </material>
     <xacro:property name = "base_width" value = "0.6" />
     <xacro:property name = "base_lenght" value = "0.4" />
