Commit message: Halledildi lakin eski halinde notlar bulunduğundan onlar da duruyor.

File: Projeler/Robot_Modelleme/robot_modelleme_ws/src/my_robot_description/urdf/main.xacro (robot description, xacro)
@@ -1,4 +1,4 @@
 <?xml version="1.0"?>
-<robot name="my_robot" xmlns:xacro = "http://www.ros.org/wiki/xacro>" > <!-- xmlns:xacro = "http://www.ros.org/wiki/xacro>" kısmı xacro kullanabilmek için.-->
+<robot name="my_robot" xmlns:xacro = "http://www.ros.org/wiki/xacro" > <!-- xmlns:xacro = "http://www.ros.org/wiki/xacro>" kısmı xacro kullanabilmek için.-->
     <xacro:include filename="my_robot.xacro"/>
     <xacro:include filename="properties.xacro"/>

File: Projeler/Robot_Modelleme/robot_modelleme_ws/src/my_robot_description/urdf/my_robot.xacro (robot description, xacro)
@@ -1,4 +1,5 @@
 <?xml version="1.0"?>
-<robot name="my_robot" xmlns:xacro = "http://www.ros.org/wiki/xacro>" > <!-- xmlns:xacro = "http://www.ros.org/wiki/xacro>" kısmı xacro kullanabilmek için.-->
+<robot name="my_robot"
+    xmlns:xacro = "http://www.ros.org/wiki/xacro">    <!-- xmlns:xacro = "http://www.ros.org/wiki/xacro>" kısmı xacro kullanabilmek için.-->
     <xacro:property name = "base_width" value = "0.6" />
     <xacro:property name = "base_lenght" value = "0.4" />
@@ -7,19 +8,37 @@
     <xacro:property name = "wheel_lenght" value = "0.05" />
     <xacro:property name = "caster_wheel_radius" value = "0.05" />
-    <xacro:macro name = "wheel_link" params = "prefix"> <!-- Tekerlek oluşturmada sadece tekar adı değiştiğinden tek tek tanımlamaktansa bir macro yazıyoruz-->
+    <xacro:macro name = "wheel_link" params = "prefix">        <!-- Tekerlek oluşturmada sadece tekar adı değiştiğinden tek tek tanımlamaktansa bir macro yazıyoruz-->
         <link name="${prefix}_wheel_link">
+            <inertial>
+                <mass value="1" />
+                <inertia ixx="1e-3" ixy="0.0" ixz="0.0" iyy="1e-3" iyz="0.0" izz="1e-3" />
+            </inertial>
             <visual>
                 <geometry>
                     <cylinder radius="${wheel_radius}" length="${wheel_lenght}"/>
                 </geometry>
-                <origin xyz="0.0 0.0 0.0" rpy="${pi/2} 0.0  0.0"/> <!-- Tekerim yatay bir biiçimde oluşuyor ve benim istediğim gibi durması için x ekseni etrafında 90 derce döndürüyorum.
-                                                                       ( kırmızı = X , Yeşil = Y , Mavi = Z)-->
+                <origin xyz="0.0 0.0 0.0" rpy="${pi/2} 0.0  0.0"/>
+                <!-- Tekerim yatay bir biiçimde oluşuyor ve benim istediğim gibi durması için x ekseni etrafında 90 derce döndürüyorum.
+                                                                     ( kırmızı = X , Yeşil = Y , Mavi = Z)-->
                 <material name="black" />
             </visual>
+            <collision>
+                <geometry>
+                    <cylinder radius="${wheel_radius}" length="${wheel_lenght}"/>
+                </geometry>
+                <origin xyz="0.0 0.0 0.0" rpy="${pi/2} 0.0  0.0"/>
+                <!-- Tekerim yatay bir biiçimde oluşuyor ve benim istediğim gibi durması için x ekseni etrafında 90 derce döndürüyorum.
+                                                                    ( kırmızı = X , Yeşil = Y , Mavi = Z)-->
+                <material name="black" />
+            </collision>
         </link>
     </xacro:macro>
     <!-- Cisim merkezi tabanın ortasında değil de tabanın üstünde olsun diye link oluşturucaz .-->
-    <link name="base_footprint" />
+    <link name="odom_link" />
     <link name="base_link">
+        <inertial>
+            <mass value="5" />
+            <inertia ixx="1e-3" ixy="0.0" ixz="0.0" iyy="1e-3" iyz="0.0" izz="1e-3" />
+        </inertial>
         <visual>
             <geometry>
@@ -29,9 +48,17 @@
             <material name="cyan" />
         </visual>
-        <!--Eylemsizlik momenti çağırma-->
-        <xacro:box_inertia m = "5.0" l = "${base_lenght}*2" w = "${base_width}" h = "${base_height}"
-                           xyz="0.0 0.0 0.0" rpy="0.0 0.0 0.0" />
+        <collision>
+            <geometry>
+                <box size="${base_width} ${base_lenght} ${base_height}"/>
+            </geometry>
+            <origin xyz="0.0 0.0 0.0" rpy="0.0 0.0 0.0"/>
+            <material name="cyan" />
+        </collision>
     </link>
     <link name="caster_wheel_link">
+        <inertial>
+            <mass value="1" />
+            <inertia ixx="1e-3" ixy="0.0" ixz="0.0" iyy="1e-3" iyz="0.0" izz="1e-3" />
+        </inertial>
         <visual>
             <geometry>
@@ -41,9 +68,16 @@
             <material name="black" />
         </visual>
+        <collision>
+            <geometry>
+                <sphere radius="${caster_wheel_radius}"/>
+            </geometry>
+            <origin xyz="0.0 0.0 0.0" rpy="0.0 0.0 0.0"/>
+            <material name="black" />
+        </collision>
     </link>
     <xacro:wheel_link prefix = "right" />
     <xacro:wheel_link prefix = "left" />
     <joint name="base_joint" type="fixed">
-        <parent link="base_footprint"/>
+        <parent link="odom_link"/>
         <child link="base_link"/>
         <origin xyz="0 0 ${(base_height/2)+wheel_radius}" rpy="0.0 0.0 0.0"/>
@@ -53,5 +87,6 @@
         <child link="right_wheel_link"/>
         <origin xyz="${-(base_width*2/6)} ${-( (base_lenght + wheel_lenght)/2)} ${-wheel_radius}" rpy="0.0 0.0 0.0"/>
-        <axis xyz="0 1 0.0"/> <!-- Cismin hangi eksenlerde dönüşüne müsaade ettiğimiz.--> <!--Duruş ayarlandıktan sonra bakıyoruz yeşil yani y ekseni etrafında dönmeli-->
+        <axis xyz="0 1 0.0"/>
+        <!-- Cismin hangi eksenlerde dönüşüne müsaade ettiğimiz.-->        <!--Duruş ayarlandıktan sonra bakıyoruz yeşil yani y ekseni etrafında dönmeli-->
         <limit lower="0.0" upper="0.0" effort="0.0" velocity="0.0"/>
     </joint>
@@ -60,5 +95,6 @@
         <child link="left_wheel_link"/>
         <origin xyz="${-(base_width*2/6)} ${( (base_lenght + wheel_lenght)/2)} ${-wheel_radius}" rpy="0.0 0.0 0.0"/>
-        <axis xyz="0 1 0.0"/> <!-- Cismin hangi eksenlerde dönüşüne müsaade ettiğimiz.--> <!--Duruş ayarlandıktan sonra bakıyoruz yeşil yani y ekseni etrafında dönmeli-->
+        <axis xyz="0 1 0.0"/>
+        <!-- Cismin hangi eksenlerde dönüşüne müsaade ettiğimiz.-->        <!--Duruş ayarlandıktan sonra bakıyoruz yeşil yani y ekseni etrafında dönmeli-->
         <limit lower="0.0" upper="0.0" effort="0.0" velocity="0.0"/>
     </joint>

File: Projeler/Robot_Modelleme/robot_modelleme_ws/src/my_robot_description/urdf/properties.xacro (robot description, xacro)
@@ -1,4 +1,4 @@
 <?xml version="1.0"?>
-<robot name="my_robot" xmlns:xacro = "http://www.ros.org/wiki/xacro>" > <!-- xmlns:xacro = "http://www.ros.org/wiki/xacro>" kısmı xacro kullanabilmek için.-->
+<robot name="my_robot" xmlns:xacro = "http://www.ros.org/wiki/xacro" > <!-- xmlns:xacro = "http://www.ros.org/wiki/xacro>" kısmı xacro kullanabilmek için.-->
 <material name="cyan">
         <color rgba="0 1 1 1"/>
@@ -7,50 +7,3 @@
         <color rgba="0 0 0 1"/>
     </material>
-    <!--Eylemsizlik momenti -->
-    <xacro:macro name = "box_inertia" params = "m l w h xyz rpy"> <!-- parametrelerim kütle ve ölçüleri.-->
-        <inertial>
-            <!-- Sırayla nesnemin origin , kütle , eylemsizliğini tanımlayacağım.-->
-            <origin xyz="${xyz}" rpy="${rpy}"/>
-            <mess value = "${m}" /> <!-- Kütle tanımladık-->
-            <inertia ixx="${(m/12) * (h*h + l*l)}" ixy="0" ixz="0"
-            iyy="${(m/12) * (w*w + l*l)}" iyz="0"
-            izz="${(m/12) * (w*w + h*h)}"/> <!--Tanımlamaları hazır olarak wikipedia da bulunuyor.-->
-            <!--
-            Eylemsizlik tensörü (moment of inertia), cismin kütlesinin dağılımına göre dönmeye karşı gösterdiği dirençtir.
-            Dikdörtgen bir kutu (box) için eylemsizlik değerleri standart fizik formülleriyle hesaplanır.
-            Bu kutunun boyutları:
-              - l: uzunluk (x ekseni yönünde)
-              - w: genişlik (y ekseni yönünde)
-              - h: yükseklik (z ekseni yönünde)
-              - m: kütle
-            Bu durumda, kutunun merkezinden geçen eksenler etrafındaki eylemsizlik momenti aşağıdaki formüllerle hesaplanır:
-            - ixx = (1/12) * m * (h² + l²)
-              -> x ekseni etrafındaki dönmeye karşı dirençtir (yükseklik ve uzunluğun karesi alınır çünkü dik eksenler onlar).
-            - iyy = (1/12) * m * (w² + l²)
-              -> y ekseni etrafındaki direnç (genişlik ve uzunluk karesi).
-            - izz = (1/12) * m * (w² + h²)
-              -> z ekseni etrafındaki direnç (genişlik ve yükseklik karesi).
-            - ixy, ixz, iyz = 0
-              -> Simetrik ve düzgün dağılımlı bir kutu için çarpraz eylemsizlik terimleri sıfırdır (off-diagonal elemanlar).
-            -->
-        </inertial>
-    </xacro:macro>
-  <xacro:macro name = "cylinder_inertia" params = "m r h xyz rpy"> <!-- parametrelerim kütle ve ölçüleri.-->
-        <inertial>
-            <origin xyz="${xyz}" rpy="${rpy}"/>
-            <mess value = "${m}" />
-            <inertia ixx="${(m/12) * (3*r*r + h*h)}" ixy="0" ixz="0"
-            iyy="${(m/12) * (3*r*r + h*h)}" iyz="0"
-            izz="${(m/2) * (r*r)}"/>
-        </inertial>
-  </xacro:macro>
-  <xacro:macro name = "sphere_inertia" params = "m r xyz rpy"> <!-- parametrelerim kütle ve ölçüleri.-->
-        <inertial>
-            <origin xyz="${xyz}" rpy="${rpy}"/>
-            <mess value = "${m}" />
-            <inertia ixx="${(2/5) * (m*r*r)}" ixy="0" ixz="0"
-            iyy="${(2/5) * (m*r*r)}" iyz="0"
-            izz="${(2/5) * (m*r*r)}"/>
-        </inertial>
-  </xacro:macro>
 </robot>
