Commit message: Temel bir robot  modelleme projesi gerçekleştirildi.

File: Projeler/Robot_Modelle/ros2_ws/install/my_robot_description/share/my_robot_description/urdf/main.xacro (robot description, xacro)
@@ -1,6 +1 @@
-<?xml version="1.0"?>
-<robot name="my_robot" xmlns:xacro = "http://www.ros.org/wiki/xacro" > <!-- xmlns:xacro = "http://www.ros.org/wiki/xacro>" kısmı xacro kullanabilmek için.-->
-    <xacro:include filename="properties.xacro"/>
-    <xacro:include filename="properties_gazebo.xacro"/>
-    <xacro:include filename="my_robot.xacro"/>
-</robot>
+/home/ibrahim/Ros_Egitim/Projeler/Robot_Modelle/ros2_ws/src/my_robot_description/urdf/main.xacro

File: Projeler/Robot_Modelle/ros2_ws/install/my_robot_description/share/my_robot_description/urdf/my_robot.xacro (robot description, xacro)
@@ -1,109 +1 @@
-<?xml version="1.0"?>
-<robot name="my_robot"
-    xmlns:xacro = "http://www.ros.org/wiki/xacro">    <!-- xmlns:xacro = "http://www.ros.org/wiki/xacro" kısmı xacro kullanabilmek için.-->
-    <xacro:property name = "base_width" value = "0.6" />
-    <xacro:property name = "base_lenght" value = "0.4" />
-    <xacro:property name = "base_height" value = "0.2" />
-    <xacro:property name = "wheel_radius" value = "0.1" />
-    <xacro:property name = "wheel_lenght" value = "0.05" />
-    <xacro:property name = "caster_wheel_radius" value = "0.05" />
-    <xacro:property name = "inertial_value_ixx" value = "1e-3" />
-    <xacro:property name = "inertial_value_iyy" value = "1e-3" />
-    <xacro:property name = "inertial_value_izz" value = "1e-3" />
-    <xacro:macro name = "wheel_link" params = "prefix">        <!-- Tekerlek oluşturmada sadece tekar adı değiştiğinden tek tek tanımlamaktansa bir macro yazıyoruz-->
-        <link name="${prefix}_wheel_link">
-            <inertial>
-                <mass value="1" />
-                <inertia ixx="${inertial_value_ixx}" ixy="0.0" ixz="0.0" iyy="${inertial_value_iyy}" iyz="0.0" izz="${inertial_value_izz}" />
-            </inertial>
-            <visual>
-                <geometry>
-                    <cylinder radius="${wheel_radius}" length="${wheel_lenght}"/>
-                </geometry>
-                <origin xyz="0.0 0.0 0.0" rpy="${pi/2} 0.0  0.0"/>
-                <!-- Tekerim yatay bir biiçimde oluşuyor ve benim istediğim gibi durması için x ekseni etrafında 90 derce döndürüyorum.
-                                                                     ( kırmızı = X , Yeşil = Y , Mavi = Z)-->
-                <material name="black" />
-            </visual>
-            <collision>
-                <geometry>
-                    <cylinder radius="${wheel_radius}" length="${wheel_lenght}"/>
-                </geometry>
-                <origin xyz="0.0 0.0 0.0" rpy="${pi/2} 0.0  0.0"/>
-                <!-- Tekerim yatay bir biiçimde oluşuyor ve benim istediğim gibi durması için x ekseni etrafında 90 derce döndürüyorum.
-                                                                    ( kırmızı = X , Yeşil = Y , Mavi = Z)-->
-                <material name="black" />
-            </collision>
-        </link>
-    </xacro:macro>
-    <!-- Cisim merkezi tabanın ortasında değil de tabanın üstünde olsun diye link oluşturucaz .-->
-    <link name="odom_link" />
-    <link name="base_link">
-        <inertial>
-            <mass value="5" />
-                <inertia ixx="${inertial_value_ixx}" ixy="0.0" ixz="0.0" iyy="${inertial_value_iyy}" iyz="0.0" izz="${inertial_value_izz}" />
-        </inertial>
-        <visual>
-            <geometry>
-                <box size="${base_width} ${base_lenght} ${base_height}"/>
-            </geometry>
-            <origin xyz="0.0 0.0 0.0" rpy="0.0 0.0 0.0"/>
-            <material name="cyan" />
-        </visual>
-        <collision>
-            <geometry>
-                <box size="${base_width} ${base_lenght} ${base_height}"/>
-            </geometry>
-            <origin xyz="0.0 0.0 0.0" rpy="0.0 0.0 0.0"/>
-            <material name="cyan" />
-        </collision>
-    </link>
-    <link name="caster_wheel_link">
-        <inertial>
-            <mass value="1" />
-            <inertia ixx="${inertial_value_ixx}" ixy="0.0" ixz="0.0" iyy="${inertial_value_iyy}" iyz="0.0" izz="${inertial_value_izz}" />
-        </inertial>
-        <visual>
-            <geometry>
-                <sphere radius="${caster_wheel_radius}"/>
-            </geometry>
-            <origin xyz="0.0 0.0 0.0" rpy="0.0 0.0 0.0"/>
-            <material name="black" />
-        </visual>
-        <collision>
-            <geometry>
-                <sphere radius="${caster_wheel_radius}"/>
-            </geometry>
-            <origin xyz="0.0 0.0 0.0" rpy="0.0 0.0 0.0"/>
-            <material name="black" />
-        </collision>
-    </link>
-    <xacro:wheel_link prefix = "right" />
-    <xacro:wheel_link prefix = "left" />
-    <joint name="base_joint" type="fixed">
-        <parent link="odom_link"/>
-        <child link="base_link"/>
-        <origin xyz="0 0 ${(base_height/2)+wheel_radius}" rpy="0.0 0.0 0.0"/>
-    </joint>
-    <joint name="base_right_wheel_joint" type="continuous">
-        <parent link="base_link"/>
-        <child link="right_wheel_link"/>
-        <origin xyz="${-(base_width*2/6)} ${-( (base_lenght + wheel_lenght)/2)} ${-wheel_radius}" rpy="0.0 0.0 0.0"/>
-        <axis xyz="0 1 0.0"/>
-        <!-- Cismin hangi eksenlerde dönüşüne müsaade ettiğimiz.-->        <!--Duruş ayarlandıktan sonra bakıyoruz yeşil yani y ekseni etrafında dönmeli-->
-        <limit lower="0.0" upper="0.0" effort="0.0" velocity="0.0"/>
-    </joint>
-    <joint name="base_left_wheel_joint" type="continuous">
-        <parent link="base_link"/>
-        <child link="left_wheel_link"/>
-        <origin xyz="${-(base_width*2/6)} ${( (base_lenght + wheel_lenght)/2)} ${-wheel_radius}" rpy="0.0 0.0 0.0"/>
-        <axis xyz="0 1 0.0"/>
-        <!-- Cismin hangi eksenlerde dönüşüne müsaade ettiğimiz.-->        <!--Duruş ayarlandıktan sonra bakıyoruz yeşil yani y ekseni etrafında dönmeli-->
-        <limit lower="0.0" upper="0.0" effort="0.0" velocity="0.0"/>
-    </joint>
-    <joint name="base_caster_wheel_joint" type="fixed">
-        <parent link="base_link"/>
-        <child link="caster_wheel_link"/>
-        <origin xyz="${base_width/4} 0 ${-(base_height/2 + caster_wheel_radius)}" rpy="0.0 0.0 0.0"/>
-    </joint>
-</robot>
+/home/ibrahim/Ros_Egitim/Projeler/Robot_Modelle/ros2_ws/src/my_robot_description/urdf/my_robot.xacro

File: Projeler/Robot_Modelle/ros2_ws/install/my_robot_description/share/my_robot_description/urdf/properties.xacro (robot description, xacro)
@@ -1,9 +1 @@
-<?xml version="1.0"?>
-<robot name="my_robot" xmlns:xacro = "http://www.ros.org/wiki/xacro" > <!-- xmlns:xacro = "http://www.ros.org/wiki/xacro>" kısmı xacro kullanabilmek için.-->
-<material name="cyan">
-        <color rgba="0 1 1 1"/>
-    </material>
-    <material name="black">
-        <color rgba="0 0 0 1"/>
-    </material>
-</robot>
+/home/ibrahim/Ros_Egitim/Projeler/Robot_Modelle/ros2_ws/src/my_robot_description/urdf/properties.xacro

File: Projeler/Robot_Modelle/ros2_ws/install/my_robot_description/share/my_robot_description/urdf/properties_gazebo.xacro (robot description, xacro)
@@ -1,6 +1 @@
-<?xml version="1.0"?>
-<robot name="my_robot" xmlns:xacro = "http://www.ros.org/wiki/xacro" > <!-- xmlns:xacro = "http://www.ros.org/wiki/xacro>" kısmı xacro kullanabilmek için.-->
-    <gazebo reference="base_link">
-        <material>Gazebo/Blue</material>
-    </gazebo>
-</robot>
+/home/ibrahim/Ros_Egitim/Projeler/Robot_Modelle/ros2_ws/src/my_robot_description/urdf/properties_gazebo.xacro

File: Projeler/Robot_Modelle/ros2_ws/src/my_robot_description/urdf/properties_gazebo.xacro (robot description, xacro)
@@ -4,3 +4,35 @@
         <material>Gazebo/Blue</material>
     </gazebo>
+    <gazebo reference="right_wheel_link">
+        <material>Gazebo/Black</material>
+    </gazebo>
+    <gazebo reference="left_wheel_link">
+        <material>Gazebo/black</material>
+    </gazebo>
+    <gazebo reference = "caster_wheel_link"> <!--Sürtünme tanımlayacağız.-->
+        <material>Gazebo/Black</material>
+        <mu1 value="0.1" />
+        <mu2 value="0.1" />
+    </gazebo>
+    <!-- gazebo ortamında hareket için .
+    https://github.com/ros-simulation/gazebo_ros_pkgs/blob/ros2/gazebo_plugins/include/gazebo_plugins/gazebo_ros_diff_drive.hpp aldık.-->
+    <gazebo>
+            <plugin name="diff_drive_controller" filename="libgazebo_ros_diff_drive.so">
+          <!-- Update rate in Hz -->
+          <update_rate>50</update_rate>
+          <!-- wheels -->
+          <left_joint>base_left_wheel_joint</left_joint>
+          <right_joint>base_right_wheel_joint</right_joint>
+          <!-- kinematics -->
+          <wheel_separation>0.45</wheel_separation> <!-- Tekerler arası mesafe-->
+          <wheel_diameter>0.2</wheel_diameter> <!--Tekerlerin çapı-->
+          <!-- output -->
+          <publish_odom>true</publish_odom>
+          <publish_odom_tf>true</publish_odom_tf>
+          <publish_wheel_tf>true</publish_wheel_tf>
+          <odometry_topic>odom</odometry_topic>
+          <odometry_frame>odom</odometry_frame>
+          <robot_base_frame>base_link</robot_base_frame>
+        </plugin>
+    </gazebo>
 </robot>
