Commit message: inertial parametreleri matematiksel formullerine göre düzenlendi

File: Projeler/Robot_Modelle/ros2_ws/src/my_robot_description/urdf/my_robot.xacro (robot description, xacro)
@@ -1,19 +1,33 @@
 <?xml version="1.0"?>
-<robot name="my_robot"
-    xmlns:xacro = "http://www.ros.org/wiki/xacro">    <!-- xmlns:xacro = "http://www.ros.org/wiki/xacro" kısmı xacro kullanabilmek için.-->
-    <xacro:property name = "base_width" value = "0.6" />
-    <xacro:property name = "base_lenght" value = "0.4" />
-    <xacro:property name = "base_height" value = "0.2" />
-    <xacro:property name = "wheel_radius" value = "0.1" />
-    <xacro:property name = "wheel_lenght" value = "0.05" />
-    <xacro:property name = "caster_wheel_radius" value = "0.05" />
-    <xacro:property name = "inertial_value_ixx" value = "1e-3" />
-    <xacro:property name = "inertial_value_iyy" value = "1e-3" />
-    <xacro:property name = "inertial_value_izz" value = "1e-3" />
-    <xacro:macro name = "wheel_link" params = "prefix">        <!-- Tekerlek oluşturmada sadece tekar adı değiştiğinden tek tek tanımlamaktansa bir macro yazıyoruz-->
+<robot name="my_robot" xmlns:xacro="http://www.ros.org/wiki/xacro">
+    <!-- === Fiziksel Parametreler === -->
+    <xacro:property name="base_width" value="0.6" />
+    <xacro:property name="base_lenght" value="0.4" />
+    <xacro:property name="base_height" value="0.2" />
+    <xacro:property name="base_mass" value="5" />
+    <xacro:property name="wheel_radius" value="0.1" />
+    <xacro:property name="wheel_lenght" value="0.05" />
+    <xacro:property name="wheel_mass" value="1" />
+    <xacro:property name="caster_wheel_radius" value="0.05" />
+    <xacro:property name="caster_mass" value="1" />
+    <!-- === Atalet Momentleri (İnertial) Hesaplamaları === -->
+    <!-- Dikdörtgen prizma için (base) -->
+    <xacro:property name="base_ixx" value="${(1/12.0)*base_mass*(base_height*base_height + base_lenght*base_lenght)}" />
+    <xacro:property name="base_iyy" value="${(1/12.0)*base_mass*(base_width*base_width + base_height*base_height)}" />
+    <xacro:property name="base_izz" value="${(1/12.0)*base_mass*(base_width*base_width + base_lenght*base_lenght)}" />
+    <!-- Silindir için (wheel) -->
+    <xacro:property name="wheel_ixx" value="${(1/12.0)*wheel_mass*(3*wheel_radius*wheel_radius + wheel_lenght*wheel_lenght)}" />
+    <xacro:property name="wheel_iyy" value="${0.5*wheel_mass*wheel_radius*wheel_radius}" />
+    <xacro:property name="wheel_izz" value="${(1/12.0)*wheel_mass*(3*wheel_radius*wheel_radius + wheel_lenght*wheel_lenght)}" />
+    <!-- Küre için (caster wheel) -->
+    <xacro:property name="caster_inertia" value="${(2/5.0)*caster_mass*caster_wheel_radius*caster_wheel_radius}" />
+    <!-- === Tekerlek Makrosu === -->
+    <xacro:macro name="wheel_link" params="prefix">
         <link name="${prefix}_wheel_link">
             <inertial>
-                <mass value="1" />
-                <inertia ixx="${inertial_value_ixx}" ixy="0.0" ixz="0.0" iyy="${inertial_value_iyy}" iyz="0.0" izz="${inertial_value_izz}" />
+                <mass value="${wheel_mass}" />
+                <inertia
+                    ixx="${wheel_ixx}" ixy="0.0" ixz="0.0"
+                    iyy="${wheel_iyy}" iyz="0.0" izz="${wheel_izz}" />
             </inertial>
             <visual>
@@ -22,6 +36,4 @@
                 </geometry>
                 <origin xyz="0.0 0.0 0.0" rpy="${pi/2} 0.0  0.0"/>
-                <!-- Tekerim yatay bir biiçimde oluşuyor ve benim istediğim gibi durması için x ekseni etrafında 90 derce döndürüyorum.
-                                                                     ( kırmızı = X , Yeşil = Y , Mavi = Z)-->
                 <material name="black" />
             </visual>
@@ -31,16 +43,16 @@
                 </geometry>
                 <origin xyz="0.0 0.0 0.0" rpy="${pi/2} 0.0  0.0"/>
-                <!-- Tekerim yatay bir biiçimde oluşuyor ve benim istediğim gibi durması için x ekseni etrafında 90 derce döndürüyorum.
-                                                                    ( kırmızı = X , Yeşil = Y , Mavi = Z)-->
                 <material name="black" />
             </collision>
         </link>
     </xacro:macro>
-    <!-- Cisim merkezi tabanın ortasında değil de tabanın üstünde olsun diye link oluşturucaz .-->
+    <!-- === Linkler === -->
     <link name="odom_link" />
     <link name="base_link">
         <inertial>
-            <mass value="5" />
-                <inertia ixx="${inertial_value_ixx}" ixy="0.0" ixz="0.0" iyy="${inertial_value_iyy}" iyz="0.0" izz="${inertial_value_izz}" />
+            <mass value="${base_mass}" />
+            <inertia
+                ixx="${base_ixx}" ixy="0.0" ixz="0.0"
+                iyy="${base_iyy}" iyz="0.0" izz="${base_izz}" />
         </inertial>
         <visual>
@@ -61,6 +73,8 @@
     <link name="caster_wheel_link">
         <inertial>
-            <mass value="1" />
-            <inertia ixx="${inertial_value_ixx}" ixy="0.0" ixz="0.0" iyy="${inertial_value_iyy}" iyz="0.0" izz="${inertial_value_izz}" />
+            <mass value="${caster_mass}" />
+            <inertia
+                ixx="${caster_inertia}" ixy="0.0" ixz="0.0"
+                iyy="${caster_inertia}" iyz="0.0" izz="${caster_inertia}" />
         </inertial>
         <visual>
@@ -81,4 +95,5 @@
     <xacro:wheel_link prefix = "right" />
     <xacro:wheel_link prefix = "left" />
+    <!-- === Eklem Tanımları === -->
     <joint name="base_joint" type="fixed">
         <parent link="odom_link"/>
