Commit message: <mu1>1.0</mu1>         <mu2>1.0</mu2> değerleri yanlış tanımlandığından robot hareket ediyordu düzeltildi ve robot duruyor.

File: Projeler/Robot_Modelle/ros2_ws/src/my_robot_description/urdf/properties_gazebo.xacro (robot description, xacro)
@@ -6,12 +6,16 @@
     <gazebo reference="right_wheel_link">
         <material>Gazebo/Black</material>
+        <!-- <mu1>1.0</mu1>
+        <mu2>1.0</mu2> -->
     </gazebo>
     <gazebo reference="left_wheel_link">
-        <material>Gazebo/black</material>
+        <material>Gazebo/Black</material>
+        <!-- <mu1>1.0</mu1>
+        <mu2>1.0</mu2> -->
     </gazebo>
     <gazebo reference = "caster_wheel_link"> <!--Sürtünme tanımlayacağız.-->
         <material>Gazebo/Black</material>
-        <mu1 value="0.1" />
-        <mu2 value="0.1" />
+        <mu1>1.0</mu1>
+        <mu2>1.0</mu2>
     </gazebo>
     <!-- gazebo ortamında hareket için .
